File: thin_sensor_XOR_PCB.kicad_pcb (KiCad board)
At the start: 2 copper layers, 35.6 x 66 mm, 39 parts, among them U1 CD4030BM96

Commit message: Added footprints, models etc
Parts:
- removed A-STOP, PROBE, TOOL, X-STOP, Y-STOP, Z-STOP: KF2EDGV-3.5-3P, thin_sensor_XOR_PCB:CONN-TH_3P-P3.50_KF2EDGV-3.5-3P
- removed ALED, PLED, YLED: SZYY0603B, thin_sensor_XOR_PCB:LED0603-R-RD_BLUE
- removed CONTROLLER, PASSTHRU: KH-RJ45-58-8P8C, thin_sensor_XOR_PCB:RJ45-TH_KH-RJ45-58-8P8C
- removed G-----P-----T, G-----X-----Y, G-----Y----NC, G-----Z-----X: Header-Male-2.54_1x3, thin_sensor_XOR_PCB:HDR-TH_3P-P2.54-V-M-1
- removed Pad_gge5686: Pad_gge5686, thin_sensor_XOR_PCB:Pad_gge5686
- removed Pad_gge6707: Pad_gge6707, thin_sensor_XOR_PCB:Pad_gge6707
- removed TLED, XLED, ZLED: SZYY0603R, thin_sensor_XOR_PCB:LED0603-R-RD
- removed USB-PROBE: KH-TYPE-C-L10-6P, thin_sensor_XOR_PCB:USB-C-TH_KH-TYPE-C-L10-6P
- added A-STOP1: Molex Microfit 3.0 43650-0315, Connector_Molex:Molex_Micro-Fit_3.0_43650-0315_1x03_P3.00mm_Vertical, F.Cu at (109.4, 71.5)
- added ALED1: SZYY0603B, LED_SMD:LED_0201_0603Metric_Pad0.64x0.40mm_HandSolder, F.Cu at (130.9, 93.4)
- added PLED1: SZYY0603B, LED_SMD:LED_0201_0603Metric_Pad0.64x0.40mm_HandSolder, F.Cu at (130.9, 95.1)
- added PROBE1: Molex Microfit 3.0 43650-0315, Connector_Molex:Molex_Micro-Fit_3.0_43650-0315_1x03_P3.00mm_Vertical, F.Cu at (109.4, 79.3)
- added RJ2: KH-RJ45-58-8P8C, thin sensor pcb custom:RJ45-TH_KH-RJ45-58-8P8C, F.Cu at (128.7, 76.1)
- added T-----P-----G1: Header-Male-2.54_1x3, Connector_PinHeader_2.54mm:PinHeader_1x03_P2.54mm_Vertical, F.Cu at (134.1, 111.0)
- added TLED1: SZYY0603R, LED_SMD:LED_0201_0603Metric_Pad0.64x0.40mm_HandSolder, F.Cu at (130.9, 96.9)
- added TOOL1: Molex Microfit 3.0 43650-0315, Connector_Molex:Molex_Micro-Fit_3.0_43650-0315_1x03_P3.00mm_Vertical, F.Cu at (109.4, 87.1)
- added USB-PROBE1: KH-TYPE-C-L10-6P, thin sensor pcb custom:USB-C-TH_KH-TYPE-C-L10-6P, F.Cu at (134.6, 90.2)
- added X-STOP1: Molex Microfit 3.0 43650-0315, Connector_Molex:Molex_Micro-Fit_3.0_43650-0315_1x03_P3.00mm_Vertical, F.Cu at (109.4, 94.9)
- added XLED1: SZYY0603R, LED_SMD:LED_0201_0603Metric_Pad0.64x0.40mm_HandSolder, F.Cu at (130.9, 98.6)
- added Y-STOP1: Molex Microfit 3.0 43650-0315, Connector_Molex:Molex_Micro-Fit_3.0_43650-0315_1x03_P3.00mm_Vertical, F.Cu at (109.4, 102.7)
- added YLED1: SZYY0603B, LED_SMD:LED_0201_0603Metric_Pad0.64x0.40mm_HandSolder, F.Cu at (130.9, 100.4)
- added Z-STOP1: Molex Microfit 3.0 43650-0315, Connector_Molex:Molex_Micro-Fit_3.0_43650-0315_1x03_P3.00mm_Vertical, F.Cu at (109.4, 110.6)
- added ZLED1: SZYY0603R, LED_SMD:LED_0201_0603Metric_Pad0.64x0.40mm_HandSolder, F.Cu at (130.9, 102.1)
- D1, D2, D3, D4, D5, D6: footprint thin_sensor_XOR_PCB:SOD-123_L2.8-W1.8-LS3.7-RD -> thin sensor pcb custom:SOD-123FL_L2.8-W1.8-LS3.7-RD
- R1, R10, R11, R2, R3, R4, R5, R6, R7, R8, R9: footprint thin_sensor_XOR_PCB:R0805 -> Resistor_SMD:R_0805_2012Metric_Pad1.20x1.40mm_HandSolder
- U1: footprint thin_sensor_XOR_PCB:SOIC-14_L8.7-W3.9-P1.27-LS6.0-BL -> thin sensor pcb custom:SOIC-14_L8.7-W3.9-P1.27-LS6.0-BL
- moved R8 39.4 mm to (126.9, 92.1), turned to 0 degrees
- moved R11 38.9 mm to (126.9, 101.0), turned to 0 degrees
- moved R2 36.2 mm to (122.1, 92.1), turned to 0 degrees
- moved R4 33.6 mm to (122.1, 98.0), turned to 0 degrees
- moved R6 33.4 mm to (122.1, 103.9), turned to 0 degrees
- moved D5 32.7 mm to (140.4, 82.1)
- moved R1 31.3 mm to (122.1, 89.2)
- moved R5 29.9 mm to (122.1, 101.0), turned to 0 degrees
- moved R3 29.2 mm to (122.1, 95.1)
- moved D4 27.3 mm to (140.4, 79.0)
- moved D6 25.2 mm to (140.4, 85.3)
- moved R10 25.0 mm to (126.9, 98.0), turned to 0 degrees
- moved D2 23.6 mm to (140.4, 72.7)
- moved D3 23.5 mm to (140.4, 75.8)
- moved R7 18.8 mm to (126.9, 89.2), turned to 0 degrees
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Connections:
- net PROBE1 renamed Probe1
- net PROBE2 renamed Probe2
- net TOOL renamed Tool
- D1 pad 1: X-STOP_3 -> Net-(D1-K)
- D2 pad 1: Y-STOP_3 -> Net-(D2-K)
- D3 pad 1: Z-STOP_3 -> Net-(D3-K)
- D4 pad 1: A-STOP_3 -> Net-(D4-K)
- D5 pad 1: TOOL_3 -> Net-(D5-K)
- D6 pad 1: PROBE_3 -> Net-(D6-K)
- R1 pad 1: XEND2 -> Xend2
- R1 pad 2: R1_2 -> Net-(XLED1--)
- R2 pad 1: YEND2 -> Yend2
- R2 pad 2: R2_2 -> Net-(YLED1--)
- R3 pad 1: ZEND2 -> Zend2
- R3 pad 2: R3_2 -> Net-(ZLED1--)
- R4 pad 1: AEND -> Aend
- R4 pad 2: R4_2 -> Net-(ALED1--)
- R5 pad 2: R5_2 -> Net-(TLED1--)
- R6 pad 2: R6_2 -> Net-(PLED1--)
- R7 pad 1: XEND1 -> Xend1
- R8 pad 1: YEND1 -> Yend1
- R9 pad 1: ZEND1 -> Zend1
- U1 pad 1: YEND1 -> unconnected-(U1-A-Pad1)
- U1 pad 10: ZEND -> unconnected-(U1-L-Pad10)
- U1 pad 11: PROBE -> Probe
- U1 pad 2: YEND2 -> unconnected-(U1-B-Pad2)
- U1 pad 3: YEND -> unconnected-(U1-J-Pad3)
- U1 pad 4: XEND -> unconnected-(U1-K-Pad4)
- U1 pad 5: XEND2 -> unconnected-(U1-C-Pad5)
- U1 pad 6: XEND1 -> unconnected-(U1-D-Pad6)
- U1 pad 8: ZEND1 -> unconnected-(U1-E-Pad8)
- U1 pad 9: ZEND2 -> unconnected-(U1-F-Pad9)
Routing:
- net VCC: track 201.6 -> 0.00 mm, vias 2 -> 0
- net GND: track 153.7 -> 0.00 mm, vias 1 -> 0
- net YEND1: track 80.9 -> 0.00 mm
- net XEND: track 66.0 -> 0.00 mm, vias 1 -> 0
- net XEND1: track 65.5 -> 0.00 mm
- net Tool: track 60.8 -> 0.00 mm
- net Probe1: track 60.1 -> 0.00 mm, vias 2 -> 0
- net SHIELD: track 60.0 -> 0.00 mm
- net AEND: track 55.3 -> 0.00 mm, vias 1 -> 0
- net ZEND1: track 51.6 -> 0.00 mm, vias 1 -> 0
- net YEND: track 49.3 -> 0.00 mm, vias 1 -> 0
- net ZEND: track 32.6 -> 0.00 mm
- net PROBE: track 31.6 -> 0.00 mm, vias 1 -> 0
- net XEND2: track 29.9 -> 0.00 mm
- net YEND2: track 29.5 -> 0.00 mm, vias 1 -> 0
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- removed copper zone on B.Cu, net GND
- removed copper zone on F.Cu, net GND
Other:
- board outline removed
- board text removed: "12V SIG GND"
- board text removed: "Jumper X,Y,Z,P to G for NC or inverted NO single sensor"
- board text removed: "Remove jumper for NO or second sensor on next PCB"
- board text removed: "V1.2 XOR"
- board text removed: "connect X+Y, Z+X, P+T for XOR combined inputs"
